File: Symétriseur et amplificateur P1 P2 P3.kicad_pcb (KiCad board)
At the start: 2 copper layers, 73 parts, among them P1 P1, P10 X2, P11 I2, P12 Y, P13 J2, P14 X3, P15 I3, P16 J3, P2 P2, P3 X1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

Commit message: update
update
Parts:
- added P17: P1, TestPoint:TestPoint_Loop_D3.80mm_Drill2.5mm, F.Cu at (99.1, 66.6)
- added P18: P1, TestPoint:TestPoint_Loop_D3.80mm_Drill2.5mm, F.Cu at (99.1, 72.7)
- added P19: P1, TestPoint:TestPoint_Loop_D3.80mm_Drill2.5mm, F.Cu at (99.1, 78.7)
Routing:
- net /VCC: track 186.5 -> 211.7 mm
- net /VSS: track 239.8 -> 253.5 mm
Other:
- board outline added: 102.2 x 94 mm
Changed lines of the file:
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@@
     )
   )
+  (footprint "TestPoint:TestPoint_Loop_D3.80mm_Drill2.5mm" (layer "F.Cu")
+    (at 99.06 78.74)
+    (descr "wire loop as test point, loop diameter 3.8mm, hole diameter 2.5mm")
+    (tags "test point wire loop bead")
+    (property "Sheetfile" "Symétriseur et amplificateur P1 P2 P3.kicad_sch")
+    (property "Sheetname" "")
+    (attr through_hole)
+    (fp_text reference "P19" (at 0.5 3.2) (layer "F.SilkS")
+        (effects (font (size 1 1) (thickness 0.15)))
+    )
+    (fp_text value "P1" (at 0 -2.8) (layer "F.Fab")
+        (effects (font (size 1 1) (thickness 0.15)))
+    )
+    (fp_text user "${REFERENCE}" (at 0.5 3.2) (layer "F.Fab")
+        (effects (font (size 1 1) (thickness 0.15)))
+    )
+    (fp_circle (center 0 0) (end 2.3 0)
+      (stroke (width 0.12) (type solid)) (fill none) (layer "F.SilkS"))
+    (fp_circle (center 0 0) (end 2.5 0)
+      (stroke (width 0.05) (type solid)) (fill none) (layer "F.CrtYd"))
+    (fp_line (start -1.9 -0.3) (end -1.9 0.3)
+      (stroke (width 0.12) (type solid)) (layer "F.Fab"))
+    (fp_line (start -1.9 0.3) (end 1.9 0.3)
+      (stroke (width 0.12) (type solid)) (layer "F.Fab"))
+    (fp_line (start 1.9 -0.3) (end -1.9 -0.3)
+      (stroke (width 0.12) (type solid)) (layer "F.Fab"))
+    (fp_line (start 1.9 0.3) (end 1.9 -0.3)
+      (stroke (width 0.12) (type solid)) (layer "F.Fab"))
+    (pad "1" thru_hole circle (at 0 0) (size 4 4) (drill 2.5) (layers "*.Cu" "*.Mask")
+      (net 3 "/VSS") (pinfunction "P1") (pintype "passive"))
+    (model "${KICAD6_3DMODEL_DIR}/TestPoint.3dshapes/TestPoint_Loop_D3.80mm_Drill2.5mm.wrl"
+      (offset (xyz 0 0 0))
+      (scale (xyz 1 1 1))
+      (rotate (xyz 0 0 0))
+    )
+  )
   (footprint "Package_TO_SOT_THT:TO-92L_Wide" (layer "F.Cu")
     (at 119.5675 104.14 -90)
@@
   )
   (footprint "TestPoint:TestPoint_Loop_D3.80mm_Drill2.5mm" (layer "F.Cu")
+    (at 99.06 72.69)
+    (descr "wire loop as test point, loop diameter 3.8mm, hole diameter 2.5mm")
+    (tags "test point wire loop bead")
+    (property "Sheetfile" "Symétriseur et amplificateur P1 P2 P3.kicad_sch")
+    (property "Sheetname" "")
+    (attr through_hole)
+    (fp_text reference "P18" (at 0.5 3.2) (layer "F.SilkS")
+        (effects (font (size 1 1) (thickness 0.15)))
+    )
+    (fp_text value "P1" (at 0 -2.8) (layer "F.Fab")
+        (effects (font (size 1 1) (thickness 0.15)))
+    )
+    (fp_text user "${REFERENCE}" (at 0.5 3.2) (layer "F.Fab")
+        (effects (font (size 1 1) (thickness 0.15)))
+    )
+    (fp_circle (center 0 0) (end 2.3 0)
+      (stroke (width 0.12) (type solid)) (fill none) (layer "F.SilkS"))
+    (fp_circle (center 0 0) (end 2.5 0)
+      (stroke (width 0.05) (type solid)) (fill none) (layer "F.CrtYd"))
+    (fp_line (start -1.9 -0.3) (end -1.9 0.3)
+      (stroke (width 0.12) (type solid)) (layer "F.Fab"))
+    (fp_line (start -1.9 0.3) (end 1.9 0.3)
+      (stroke (width 0.12) (type solid)) (layer "F.Fab"))
+    (fp_line (start 1.9 -0.3) (end -1.9 -0.3)
+      (stroke (width 0.12) (type solid)) (layer "F.Fab"))
+    (fp_line (start 1.9 0.3) (end 1.9 -0.3)
+      (stroke (width 0.12) (type solid)) (layer "F.Fab"))
+    (pad "1" thru_hole circle (at 0 0) (size 4 4) (drill 2.5) (layers "*.Cu" "*.Mask")
+      (net 2 "GND") (pinfunction "P1") (pintype "passive"))
+    (model "${KICAD6_3DMODEL_DIR}/TestPoint.3dshapes/TestPoint_Loop_D3.80mm_Drill2.5mm.wrl"
+      (offset (xyz 0 0 0))
+      (scale (xyz 1 1 1))
+      (rotate (xyz 0 0 0))
+    )
+  )
+  (footprint "TestPoint:TestPoint_Loop_D3.80mm_Drill2.5mm" (layer "F.Cu")
     (at 167.64 87.63)
     (descr "wire loop as test point, loop diameter 3.8mm, hole diameter 2.5mm")
@@
     )
   )
+  (footprint "TestPoint:TestPoint_Loop_D3.80mm_Drill2.5mm" (layer "F.Cu")
+    (at 99.06 66.64)
+    (descr "wire loop as test point, loop diameter 3.8mm, hole diameter 2.5mm")
+    (tags "test point wire loop bead")
+    (property "Sheetfile" "Symétriseur et amplificateur P1 P2 P3.kicad_sch")
+    (property "Sheetname" "")
+    (attr through_hole)
+    (fp_text reference "P17" (at 0.5 3.2) (layer "F.SilkS")
+        (effects (font (size 1 1) (thickness 0.15)))
+    )
+    (fp_text value "P1" (at 0 -2.8) (layer "F.Fab")
+        (effects (font (size 1 1) (thickness 0.15)))
+    )
+    (fp_text user "${REFERENCE}" (at 0.5 3.2) (layer "F.Fab")
+        (effects (font (size 1 1) (thickness 0.15)))
+    )
+    (fp_circle (center 0 0) (end 2.3 0)
+      (stroke (width 0.12) (type solid)) (fill none) (layer "F.SilkS"))
+    (fp_circle (center 0 0) (end 2.5 0)
+      (stroke (width 0.05) (type solid)) (fill none) (layer "F.CrtYd"))
+    (fp_line (start -1.9 -0.3) (end -1.9 0.3)
+      (stroke (width 0.12) (type solid)) (layer "F.Fab"))
+    (fp_line (start -1.9 0.3) (end 1.9 0.3)
+      (stroke (width 0.12) (type solid)) (layer "F.Fab"))
+    (fp_line (start 1.9 -0.3) (end -1.9 -0.3)
+      (stroke (width 0.12) (type solid)) (layer "F.Fab"))
+    (fp_line (start 1.9 0.3) (end 1.9 -0.3)
+      (stroke (width 0.12) (type solid)) (layer "F.Fab"))
+    (pad "1" thru_hole circle (at 0 0) (size 4 4) (drill 2.5) (layers "*.Cu" "*.Mask")
+      (net 4 "/VCC") (pinfunction "P1") (pintype "passive"))
+    (model "${KICAD6_3DMODEL_DIR}/TestPoint.3dshapes/TestPoint_Loop_D3.80mm_Drill2.5mm.wrl"
+      (offset (xyz 0 0 0))
+      (scale (xyz 1 1 1))
+      (rotate (xyz 0 0 0))
+    )
+  )
   (footprint "Resistor_THT:R_Axial_DIN0207_L6.3mm_D2.5mm_P10.16mm_Horizontal" (layer "F.Cu")
     (at 111.76 71.12 -90)
@@
   (gr_line (start 196.85 44.45) (end 196.85 138.43)
     (stroke (width 0.15) (type default)) (layer "Eco2.User"))
+  (gr_line (start 95.25 138.43) (end 95.25 44.45)
+    (stroke (width 0.05) (type default)) (layer "Edge.Cuts"))
+  (gr_line (start 95.25 44.45) (end 196.85 44.45)
+    (stroke (width 0.05) (type default)) (layer "Edge.Cuts"))
+  (gr_line (start 196.85 44.45) (end 196.85 138.43)
+    (stroke (width 0.05) (type default)) (layer "Edge.Cuts"))
+  (gr_line (start 196.85 138.43) (end 94.615 138.43)
+    (stroke (width 0.05) (type default)) (layer "Edge.Cuts"))
   (segment (start 123.19 55.88) (end 124.46 54.61) (width 1.27) (layer "B.Cu") (net 1))
   (segment (start 124.46 58.42) (end 124.46 53.22) (width 1.27) (layer "B.Cu") (net 1))
@@
   (segment (start 191.77 127) (end 194.31 124.46) (width 1.27) (layer "F.Cu") (net 3))
   (segment (start 130.175 81.28) (end 140.97 81.28) (width 1.27) (layer "F.Cu") (net 3))
+  (segment (start 99.06 78.74) (end 102.235 78.74) (width 1.27) (layer "F.Cu") (net 3))
   (segment (start 181.61 127) (end 191.77 127) (width 1.27) (layer "F.Cu") (net 3))
   (segment (start 172.72 80.01) (end 172.72 81.28) (width 1.27) (layer "F.Cu") (net 3))
@@
   (segment (start 111.76 83.82) (end 113.03 85.09) (width 1.27) (layer "F.Cu") (net 3))
   (segment (start 194.31 124.46) (end 194.31 90.17) (width 1.27) (layer "F.Cu") (net 3))
+  (segment (start 104.775 81.28) (end 111.76 81.28) (width 1.27) (layer "F.Cu") (net 3))
   (segment (start 128.27 81.28) (end 130.175 81.28) (width 1.27) (layer "F.Cu") (net 3))
   (segment (start 124.46 85.09) (end 128.27 81.28) (width 1.27) (layer "F.Cu") (net 3))
@@
   (segment (start 189.23 85.09) (end 176.53 85.09) (width 1.27) (layer "F.Cu") (net 3))
   (segment (start 143.805 78.445) (end 171.155 78.445) (width 1.27) (layer "F.Cu") (net 3))
+  (segment (start 102.235 78.74) (end 104.775 81.28) (width 1.27) (layer "F.Cu") (net 3))
   (segment (start 140.97 81.28) (end 143.805 78.445) (width 1.27) (layer "F.Cu") (net 3))
   (segment (start 194.31 90.17) (end 189.23 85.09) (width 1.27) (layer "F.Cu") (net 3))
@@
   (segment (start 158.75 62.23) (end 157.48 60.96) (width 1.27) (layer "B.Cu") (net 4))
   (segment (start 157.48 60.96) (end 152.4 60.96) (width 1.27) (layer "B.Cu") (net 4))
+  (segment (start 119.38 60.96) (end 121.92 60.96) (width 1.27) (layer "B.Cu") (net 4))
   (segment (start 187.96 88.9) (end 184.15 88.9) (width 1.27) (layer "B.Cu") (net 4))
+  (segment (start 102.905 66.64) (end 105.41 64.135) (width 1.27) (layer "B.Cu") (net 4))
+  (segment (start 116.205 64.135) (end 119.38 60.96) (width 1.27) (layer "B.Cu") (net 4))
+  (segment (start 105.41 64.135) (end 116.205 64.135) (width 1.27) (layer "B.Cu") (net 4))
+  (segment (start 99.06 66.64) (end 102.905 66.64) (width 1.27) (layer "B.Cu") (net 4))
   (segment (start 111.76 88.9) (end 121.92 88.9) (width 1.27) (layer "B.Cu") (net 4))
   (segment (start 184.15 88.9) (end 173.99 88.9) (width 1.27) (layer "B.Cu") (net 4))
@@
   (segment (start 175.26 134.62) (end 179.07 134.62) (width 1.27) (layer "B.Cu") (net 38))
   (zone (net 2) (net_name "GND") (layers "F&B.Cu") (hatch edge 0.5)
+    (priority 1)
+    (connect_pads (clearance 0.5))
+    (min_thickness 0.25) (filled_areas_thickness no)
+    (fill yes (thermal_gap 0.5) (thermal_bridge_width 0.5))
+    (polygon
+      (pts
+        (xy 95.25 44.45)
+        (xy 196.85 44.45)
+        (xy 196.85 138.43)
+        (xy 95.25 138.43)
+      )
+    )
+  )
+  (zone (net 2) (net_name "GND") (layers "F&B.Cu") (hatch edge 0.5)
     (connect_pads (clearance 0.5))
