File: Symétriseur et amplificateur P1 P2 P3.kicad_sch (KiCad schematic)
At the start: 69 parts, among them P10 P2, P11 X1, P12 P3, P13 X2, P14 X1, P15 I1, P16 X3, P17 J1, P18 X2, P19 I2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

Commit message: update
update
Parts:
- added P8 (x3): P1, TestPoint:TestPoint_Loop_D3.80mm_Drill2.5mm, symbol carte_num-rescue:CONN_01X01
Connections:
- net GND: now also P8.1 (P1)
- net VCC: now also P8.1 (P1)
- net VSS: now also P8.1 (P1)
Changed lines of the file:
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@@
     (effects (font (size 1.524 1.524)) (justify left bottom))
+  )
+  (label "VSS" (at 200.66 54.61 0) (fields_autoplaced)
+    (effects (font (size 1.27 1.27)) (justify left bottom))
+  )
+  (label "VCC" (at 200.66 39.37 0) (fields_autoplaced)
+    (effects (font (size 1.27 1.27)) (justify left bottom))
   )
   (label "VSS" (at 124.46 154.94 0) (fields_autoplaced)
@@
     (effects (font (size 1.524 1.524)) (justify left bottom))
   )
+  (label "GND" (at 200.66 46.99 0) (fields_autoplaced)
+    (effects (font (size 1.27 1.27)) (justify left bottom))
+  )
   (label "VCC" (at 128.905 84.455 0) (fields_autoplaced)
     (effects (font (size 1.524 1.524)) (justify left bottom))
@@
     )
   )
+  (symbol (lib_id "carte_num-rescue:CONN_01X01") (at 195.58 54.61 180) (unit 1)
+    (in_bom yes) (on_board yes) (dnp no)
+    (property "Reference" "P8" (at 195.58 57.15 0)
+      (effects (font (size 1.27 1.27)))
+    )
+    (property "Value" "P1" (at 195.58 52.705 0)
+      (effects (font (size 1.27 1.27)))
+    )
+    (property "Footprint" "TestPoint:TestPoint_Loop_D3.80mm_Drill2.5mm" (at 195.58 54.61 0)
+      (effects (font (size 1.27 1.27)) hide)
+    )
+    (property "Datasheet" "" (at 195.58 54.61 0)
+      (effects (font (size 1.27 1.27)))
+    )
+    (pin "1")
+    (instances
+      (project "Kaneda-SP10"
+        (path "/7a82d427-fea7-4249-9c5a-59087a103697"
+          (reference "P8") (unit 1)
+        )
+      )
+      (project "Symétriseur et amplificateur P1 P2 P3"
+        (path "/7d9ed54d-3fc1-4a66-a75d-5cfb3bd66c6d"
+          (reference "P19") (unit 1)
+        )
+      )
+    )
+  )
   (symbol (lib_id "carte_num-rescue:CONN_01X01") (at 146.05 91.44 90) (unit 1)
     (in_bom yes) (on_board yes) (dnp no)
@@
     )
   )
+  (symbol (lib_id "carte_num-rescue:CONN_01X01") (at 195.58 46.99 180) (unit 1)
+    (in_bom yes) (on_board yes) (dnp no)
+    (property "Reference" "P8" (at 195.58 49.53 0)
+      (effects (font (size 1.27 1.27)))
+    )
+    (property "Value" "P1" (at 195.58 45.085 0)
+      (effects (font (size 1.27 1.27)))
+    )
+    (property "Footprint" "TestPoint:TestPoint_Loop_D3.80mm_Drill2.5mm" (at 195.58 46.99 0)
+      (effects (font (size 1.27 1.27)) hide)
+    )
+    (property "Datasheet" "" (at 195.58 46.99 0)
+      (effects (font (size 1.27 1.27)))
+    )
+    (pin "1")
+    (instances
+      (project "Kaneda-SP10"
+        (path "/7a82d427-fea7-4249-9c5a-59087a103697"
+          (reference "P8") (unit 1)
+        )
+      )
+      (project "Symétriseur et amplificateur P1 P2 P3"
+        (path "/7d9ed54d-3fc1-4a66-a75d-5cfb3bd66c6d"
+          (reference "P18") (unit 1)
+        )
+      )
+    )
+  )
   (symbol (lib_id "carte_num-rescue:C") (at 64.135 71.12 270) (mirror x) (unit 1)
     (in_bom yes) (on_board yes) (dnp no)
@@
         )
       )
+    )
+  )
+  (symbol (lib_id "carte_num-rescue:CONN_01X01") (at 195.58 39.37 180) (unit 1)
+    (in_bom yes) (on_board yes) (dnp no)
+    (property "Reference" "P8" (at 195.58 41.91 0)
+      (effects (font (size 1.27 1.27)))
+    )
+    (property "Value" "P1" (at 195.58 37.465 0)
+      (effects (font (size 1.27 1.27)))
+    )
+    (property "Footprint" "TestPoint:TestPoint_Loop_D3.80mm_Drill2.5mm" (at 195.58 39.37 0)
+      (effects (font (size 1.27 1.27)) hide)
+    )
+    (property "Datasheet" "" (at 195.58 39.37 0)
+      (effects (font (size 1.27 1.27)))
+    )
+    (pin "1")
+    (instances
+      (project "Kaneda-SP10"
+        (path "/7a82d427-fea7-4249-9c5a-59087a103697"
+          (reference "P8") (unit 1)
+        )
+      )
+      (project "Symétriseur et amplificateur P1 P2 P3"
+        (path "/7d9ed54d-3fc1-4a66-a75d-5cfb3bd66c6d"
+          (reference "P17") (unit 1)
+        )
+      )
